File: Pehlivan VCU.kicad_sch (KiCad schematic)
At the start: 57 parts, among them J1 PWR_IN, J2 DEBUG, J3 SD_CARD MODULE, J4 Headlights, J5 Nextion, J6 LORA, J7 Blinker, J8 CAN, J9 Stop, U1 L7805, U2 STM32G431C8Tx, U3 LM1117MP-3.3, U4 BTS432, U5 BTS432, U6 BTS432, U7 BTS432, U8 TJA1051T-3, U9 BTS432, Y1 16MHz 18pF

Commit message: rev.0.1
Parts:
- H1, H2, H3, H4: footprint (none) -> MountingHole:MountingHole_2.7mm_M2.5
Changed lines of the file:
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@@
 			)
 		)
-		(property "Footprint" ""
+		(property "Footprint" "MountingHole:MountingHole_2.7mm_M2.5"
 			(at 223.52 63.5 0)
 			(hide yes)
@@
 			)
 		)
-		(property "Footprint" ""
+		(property "Footprint" "MountingHole:MountingHole_2.7mm_M2.5"
 			(at 204.47 63.5 0)
 			(hide yes)
@@
 			)
 		)
-		(property "Footprint" ""
+		(property "Footprint" "MountingHole:MountingHole_2.7mm_M2.5"
 			(at 245.11 63.5 0)
 			(hide yes)
@@
 			)
 		)
-		(property "Footprint" ""
+		(property "Footprint" "MountingHole:MountingHole_2.7mm_M2.5"
 			(at 265.43 63.5 0)
 			(hide yes)

Commit message: changes
Parts:
- removed BT1: Battery_Cell, Battery:BatteryHolder_Keystone_1060_1x2032, symbol Device:Battery_Cell
- removed C1: 100nF, Capacitor_SMD:C_0805_2012Metric_Pad1.18x1.45mm_HandSolder, symbol Device:C
- removed C4, C5: 26pF, Capacitor_SMD:C_0603_1608Metric_Pad1.08x0.95mm_HandSolder, symbol Device:C
- removed U2: STM32G431C8Tx, Package_QFP:LQFP-48_7x7mm_P0.5mm, symbol MCU_ST_STM32G4:STM32G431C8Tx
- removed Y1: 16MHz 18pF, Crystal:Crystal_SMD_3225-4Pin_3.2x2.5mm_HandSoldering, symbol Device:Crystal_GND24
- added C17, C19: 100nF, Capacitor_SMD:C_0805_2012Metric_Pad1.18x1.45mm_HandSolder, symbol Device:C
- added C20, C22: 26pF, Capacitor_SMD:C_0603_1608Metric_Pad1.08x0.95mm_HandSolder, symbol Device:C
- added D1, D10, D2, D9: LED, LED_SMD:LED_1206_3216Metric_Pad1.42x1.75mm_HandSolder, symbol Device:LED
- added D3: SMAJ16CA, Diode_SMD:D_SMA, symbol Diode:SMAJ16CA
- added J7: IN1, TerminalBlock_Phoenix:TerminalBlock_Phoenix_MKDS-1,5-3-5.08_1x03_P5.08mm_Horizontal, symbol Connector_Generic:Conn_01x03
- added J8: IN2, TerminalBlock_Phoenix:TerminalBlock_Phoenix_MKDS-1,5-3-5.08_1x03_P5.08mm_Horizontal, symbol Connector_Generic:Conn_01x03
- added J9: GND, TerminalBlock_Phoenix:TerminalBlock_Phoenix_MKDS-1,5-3-5.08_1x03_P5.08mm_Horizontal, symbol Connector_Generic:Conn_01x03
- added Q4, Q5: BC817, Package_TO_SOT_SMD:SOT-23, symbol Transistor_BJT:BC817
- added R16, R17, R2: 1k, Resistor_SMD:R_0805_2012Metric, symbol Device:R
- added R19, R20: 4.7K, Resistor_SMD:R_0805_2012Metric_Pad1.20x1.40mm_HandSolder, symbol Device:R
- added U10: STM32G431C8Tx, Package_QFP:LQFP-48_7x7mm_P0.5mm, symbol MCU_ST_STM32G4:STM32G431C8Tx
- added Y2: 16MHz 18pF, Crystal:Crystal_SMD_3225-4Pin_3.2x2.5mm_HandSoldering, symbol Device:Crystal_GND24
- H1, H2, H3, H4: footprint MountingHole:MountingHole_2.7mm_M2.5 -> MountingHole:MountingHole_2.7mm_M2.5_DIN965_Pad
- R1: value 10k -> 1k; footprint Resistor_SMD:R_0805_2012Metric_Pad1.20x1.40mm_HandSolder -> Resistor_SMD:R_0805_2012Metric
- R10: renamed from R3; footprint Resistor_SMD:R_1210_3225Metric_Pad1.30x2.65mm_HandSolder -> Resistor_SMD:R_0805_2012Metric
- R11: renamed from R5; footprint Resistor_SMD:R_1210_3225Metric_Pad1.30x2.65mm_HandSolder -> Resistor_SMD:R_0805_2012Metric
- R13: renamed from R6; footprint Resistor_SMD:R_1210_3225Metric_Pad1.30x2.65mm_HandSolder -> Resistor_SMD:R_0805_2012Metric
- R14: renamed from R8; footprint Resistor_SMD:R_1210_3225Metric_Pad1.30x2.65mm_HandSolder -> Resistor_SMD:R_0805_2012Metric
- R15: renamed from R11; footprint Resistor_SMD:R_1210_3225Metric_Pad1.30x2.65mm_HandSolder -> Resistor_SMD:R_0805_2012Metric
- R6: renamed from R4; footprint Resistor_SMD:R_1210_3225Metric_Pad1.30x2.65mm_HandSolder -> Resistor_SMD:R_0805_2012Metric
- R7: footprint Resistor_SMD:R_1210_3225Metric_Pad1.30x2.65mm_HandSolder -> Resistor_SMD:R_0805_2012Metric
- R8: renamed from R9; footprint Resistor_SMD:R_1210_3225Metric_Pad1.30x2.65mm_HandSolder -> Resistor_SMD:R_0805_2012Metric
- R9: renamed from R12; footprint Resistor_SMD:R_1210_3225Metric_Pad1.30x2.65mm_HandSolder -> Resistor_SMD:R_0805_2012Metric
- renumbered C3 to C1, C6 to C10, C7 to C11, C8 to C12, C19 to C13, C10 to C14, C16 to C15, C18 to C16, C14 to C18, C9 to C2, C12 to C3, C13 to C4, C15 to C5, C17 to C6, C20 to C7, C11 to C8, C2 to C9, J4 to J10, J7 to J11, J9 to J12, J5 to J3, J8 to J4, J3 to J5, R13 to R3, R10 to R4, R2 to R5, U3 to U2, U8 to U3, U4 to U5, U5 to U6, U6 to U7, U7 to U8
Connections:
- net UART3_TX is gone; now on net UART2_TX: J6.3 (Pin_3)
- net +3V3: now also C17.1, Q4.3 (C), Q5.3 (C), R2.2, U10.1 (VBAT), U10.21 (VDDA), U10.24 (VDD), U10.36 (VDD), U10.48 (VDD)
- net +5V: now also J3.1 (Pin_1), R1.2; no longer J3.4 (Pin_4)
- net Brake_FAULT: now also U10.33 (PA11)
- net FDCAN_RX: now also U10.46 (PB9)
- net FDCAN_TX: now also U10.45 (PB8)
- net F_BrakeLights: now also U10.34 (PA12)
- net F_Headlights: now also U10.28 (PB14)
- net GND: now also J3.4 (Pin_4), C17.2, C19.2, C20.2, C22.1, D1.1 (K), D10.1 (K), D2.1 (K), D3.2 (A2), D9.1 (K), J8.3 (Pin_3), J9.1 (Pin_1), J9.2 (Pin_2), J9.3 (Pin_3), U10.19 (VSSA), U10.23 (VSS), U10.35 (VSS), U10.47 (VSS), Y2.2 (G), Y2.4 (G); no longer J3.1 (Pin_1), R1.1
- net HSE_IN: now also C20.1, U10.5 (PF0), Y2.1
- net HSE_OUT: now also C22.2, U10.6 (PF1), Y2.3
- net L_BL_FAULT: now also U10.32 (PA10)
- net L_Blinker: now also U10.31 (PA9)
- net L_HL_FAULT: now also U6.4 (ST), U10.26 (PB12); no longer U5.4 (ST)
- net L_HL_OUT: now also J10.1 (Pin_1), U6.5 (OUT); no longer J10.3 (Pin_3), U5.5 (OUT)
- net NRST: now also C19.1, U10.7 (PG10)
- net R_BL_FAULT: now also U10.29 (PB15)
- net R_Blinker: now also U10.30 (PA8)
- net R_HL_FAULT: now also U5.4 (ST), U10.27 (PB13); no longer U6.4 (ST)
- net R_HL_OUT: now also J10.3 (Pin_3), U5.5 (OUT); no longer J10.1 (Pin_1), U6.5 (OUT)
- net SPICK: now also U10.13 (PA5)
- net SPIMISO: now also U10.14 (PA6)
- net SPIMOSI: now also U10.15 (PA7)
- net SPI_CS: now also U10.16 (PB0)
- net SWDCLK: now also U10.38 (PA14)
- net SWDIO: now also U10.37 (PA13)
- net UART2_RX: now also J6.2 (Pin_2), U10.40 (PB3); no longer J3.2 (Pin_2)
- net UART2_TX: now also R20.1, U10.41 (PB4); no longer J3.3 (Pin_3)
- net VCC: now also D3.1 (A1)
- net VREF: now also U10.20 (VREF+)
- net CANN: now reaches J4.1 (Pin_1), R4.2, U3.6 (CANL)
- net CANP: now reaches J4.2 (Pin_2), R4.1, U3.7 (CANH)
- net at R10.2: now also U6.2 (IN); no longer U5.2 (IN)
- net at R11.1: now also U5.2 (IN); no longer U6.2 (IN)
- removed net UART3_RX: J6.2 (Pin_2), R1.2
- new net: Q4.1 (B), R19.2
- new net: Q5.1 (B), R20.2
- new net: Q5.2 (E), R17.1
- new net: D9.2 (A), R16.2
- new net: D1.2 (A), R1.1
- new net: D10.2 (A), R17.2
- new net: Q4.2 (E), R16.1
- new net: D2.2 (A), R2.1
- new net Brake_IN: J8.2 (Pin_2), U10.12 (PA4)
- new net Hazards_IN: J7.3 (Pin_3), U10.10 (PA2)
- new net Headlights_IN: J8.1 (Pin_1), U10.11 (PA3)
- new net Left_Signal_IN: J7.1 (Pin_1), U10.8 (PA0)
- new net Right_Signal_IN: J7.2 (Pin_2), U10.9 (PA1)
- new net UART1_RX: J3.2 (Pin_2), U10.43 (PB6)
- new net UART1_TX: J3.3 (Pin_3), R19.1, U10.44 (PB7)
- no-connect marks 13 -> 9
Other:
- note added: "--- HSE CRYSTAL LOAD CAPACITANCE CALCULATION --- Formula: Cl = ((C1 * C2) / (C1 + C2)) + Cs Given: - Cl (Crystal Load Capacitance) = 18 pF (Raltron RH100) - C1 = C2 = Cx (Symmetric Load Capacitors) - Cs (Stray/PCB Capacitance) ~= 5 pF (Assumed) Calculation: 18 pF = (Cx / 2) + 5 pF 13 pF = Cx / 2 Cx = 26 pF (Standard 22pF or 27pF can be used) ------------------------------------------------"
- note added: "Not(TR): Eğer HSI (Dahili Yüksek Hızlı Osilatör) kullanılacaksa, Y1 kristalinin karta lehimlenmesine gerek yoktur. Ancak, dış kaynaklardan gelen aşırı EMI (elektromanyetik gürültü) veya yüksek sıcaklık nedeniyle kararlılık/stabilizasyon bozulursa, Y1 (harici kristal) kullanılmalıdır! Bu durumda yazılım güncellemesi yapılması gerekir. NOTE(ENG): If HSI (Internal High-Speed Oscillator) is used, sol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"
- note removed: "Cl = (C1xC2 / C1+C2)+ Cs C1 = C2 = Cx Cs = 5pF 18 = (Cx/2)+ 5 Cx = 26pF"
- note removed: "Note: HSI kullanılacaksa X1'i, takmaya gerek kalmıyor. Stabilizasyon bozulursa X1 Takılabilir."
- moved on the sheet: C13, C15, C16, C18, C5, C6, C7, H1, H2, H3, H4, J10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
