File: Pehlivan VCU.kicad_sch (KiCad schematic)
At the start: 72 parts, among them J1 PWR_IN, J10 Headlights, J11 Blinker, J12 Stop, J2 DEBUG, J3 Nextion, J4 CAN, J5 SD_CARD MODULE, J6 LORA, J7 IN1, J8 IN2, J9 GND, Q4 BC817, Q5 BC817, U1 L7805, U10 STM32G431C8Tx, U2 LM1117MP-3.3, U3 TJA1051T-3, U5 BTS432, U6 BTS432, U7 BTS432, U8 BTS432, U9 BTS432, Y2 16MHz 18pF

Commit message: changes
Parts:
- removed C22: 26pF, Capacitor_SMD:C_0603_1608Metric_Pad1.08x0.95mm_HandSolder, symbol Device:C
- removed D3: SMAJ16CA, Diode_SMD:D_SMA, symbol Diode:SMAJ16CA
- removed U2: LM1117MP-3.3, Package_TO_SOT_SMD:SOT-223-3_TabPin2, symbol Regulator_Linear:LM1117MP-3.3
- removed Y2: 16MHz 18pF, Crystal:Crystal_SMD_3225-4Pin_3.2x2.5mm_HandSoldering, symbol Device:Crystal_GND24
- added C21: 10uF, Capacitor_THT:C_Radial_D5.0mm_H5.0mm_P2.00mm, symbol Device:C_Polarized
- added J13: LORA, Connector_PinSocket_2.54mm:PinSocket_1x04_P2.54mm_Horizontal, symbol Connector_Generic:Conn_01x04
- added TP1, TP2, TP3, TP4, TP5, TP6, TP7, TP8, TP9: TestPoint, TestPoint:TestPoint_Pad_D1.0mm, symbol Connector:TestPoint
- added U2: XC6206P332MR, Package_TO_SOT_SMD:SOT-23-3, symbol Regulator_Linear:XC6206PxxxMR
- C10, C11, C14, C17, C9: footprint Capacitor_SMD:C_0805_2012Metric_Pad1.18x1.45mm_HandSolder -> Capacitor_SMD:C_0603_1608Metric
- C20: value 26pF -> 100nF; footprint Capacitor_SMD:C_0603_1608Metric_Pad1.08x0.95mm_HandSolder -> Capacitor_SMD:C_0805_2012Metric_Pad1.18x1.45mm_HandSolder
- J6: footprint Connector_PinSocket_2.54mm:PinSocket_1x04_P2.54mm_Vertical -> Connector_PinSocket_2.54mm:PinSocket_1x04_P2.54mm_Horizontal
- R5: footprint Resistor_SMD:R_0805_2012Metric_Pad1.20x1.40mm_HandSolder -> Resistor_SMD:R_0603_1608Metric_Pad0.98x0.95mm_HandSolder
Connections:
- net +3V3: now also U2.2 (VO)
- net +5V: now also C20.2, C21.1, J13.4 (Pin_4), U2.3 (VI)
- net Brake_IN: now also TP9.1
- net F_BrakeLights: now also TP4.1
- net F_Headlights: now also TP1.1
- net GND: now also C20.1, C21.2, J13.1 (Pin_1), U2.1 (GND); no longer C20.2
- net Hazards_IN: now also TP7.1
- net Headlights_IN: now also TP8.1
- net L_Blinker: now also TP2.1
- net Left_Signal_IN: now also TP5.1
- net R_Blinker: now also TP3.1
- net Right_Signal_IN: now also TP6.1
- net UART3_TX: now reaches U10.22 (PB10)
- net UART3_TX: now also J13.3 (Pin_3)
- net UART3_RX: now reaches U10.25 (PB11)
- net UART3_RX: now also J13.2 (Pin_2)
- net HSE_IN: no longer names the net of U10.5 (PF0)
- net HSE_IN: no longer C20.1
- net HSE_OUT: no longer names the net of U10.6 (PF1)
Other:
- company: (none) -> Pehlivan Team
- title: PehlivanVCU -> Vehicle Control Unit
- moved on the sheet: J7, J8, J9
